File: tutorial-77.kicad_pcb (KiCad board)
At the start: 2 copper layers, 25 x 25 mm, 7 parts, among them J1 Conn_01x03_Pin, U1 ATtiny85-20S

Commit message: オートルーターを使用plan_a
Routing:
- net GND: track 0.00 -> 23.7 mm
- net Net-(J1-Pin_1): track 0.00 -> 9.62 mm
- net VCC: track 0.00 -> 7.43 mm
- net /INPUT: track 0.00 -> 5.97 mm
- net Net-(D1-A): track 0.00 -> 3.92 mm
- net Net-(D1-K): track 0.00 -> 1.94 mm
Changed lines of the file:
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@@
 		)
+	)
+	(segment
+		(start 125.715 120.955)
+		(end 123.885 120.955)
+		(width 0.1524)
+		(layer "F.Cu")
+		(net "Net-(D1-K)")
+	)
+	(segment
+		(start 123.885 120.955)
+		(end 123.81 121.03)
+		(width 0.1524)
+		(layer "F.Cu")
+		(net "Net-(D1-K)")
+	)
+	(segment
+		(start 128.0714 120.145998)
+		(end 128.295998 119.9214)
+		(width 0.1524)
+		(layer "F.Cu")
+		(net "GND")
+	)
+	(segment
+		(start 129.929002 119.9214)
+		(end 130.8209 120.813298)
+		(width 0.1524)
+		(layer "F.Cu")
+		(net "GND")
+	)
+	(segment
+		(start 130.8209 121.319101)
+		(end 130.8209 122.3683)
+		(width 0.1524)
+		(layer "F.Cu")
+		(net "GND")
+	)
+	(segment
+		(start 123.81 119.205)
+		(end 124.750998 120.145998)
+		(width 0.1524)
+		(layer "F.Cu")
+		(net "GND")
+	)
+	(segment
+		(start 128.295998 119.9214)
+		(end 129.929002 119.9214)
+		(width 0.1524)
+		(layer "F.Cu")
+		(net "GND")
+	)
+	(segment
+		(start 130.8209 125.5809)
+		(end 130.8209 122.3683)
+		(width 0.1524)
+		(layer "F.Cu")
+		(net "GND")
+	)
+	(segment
+		(start 132.7 127.46)
+		(end 130.8209 125.5809)
+		(width 0.1524)
+		(layer "F.Cu")
+		(net "GND")
+	)
+	(segment
+		(start 136.2875 116.665)
+		(end 135.475001 116.665)
+		(width 0.1524)
+		(layer "F.Cu")
+		(net "GND")
+	)
+	(segment
+		(start 130.8209 120.813298)
+		(end 130.8209 122.3683)
+		(width 0.1524)
+		(layer "F.Cu")
+		(net "GND")
+	)
+	(segment
+		(start 135.475001 116.665)
+		(end 130.8209 121.319101)
+		(width 0.1524)
+		(layer "F.Cu")
+		(net "GND")
+	)
+	(segment
+		(start 124.750998 120.145998)
+		(end 128.0714 120.145998)
+		(width 0.1524)
+		(layer "F.Cu")
+		(net "GND")
+	)
+	(segment
+		(start 129.1125 120.475)
+		(end 129.1125 122.3517)
+		(width 0.1524)
+		(layer "F.Cu")
+		(net "VCC")
+	)
+	(segment
+		(start 130.16 127.46)
+		(end 129.0959 126.3959)
+		(width 0.1524)
+		(layer "F.Cu")
+		(net "VCC")
+	)
+	(segment
+		(start 129.1125 122.3517)
+		(end 129.0959 122.3683)
+		(width 0.1524)
+		(layer "F.Cu")
+		(net "VCC")
+	)
+	(segment
+		(start 129.0959 126.3959)
+		(end 129.0959 122.3683)
+		(width 0.1524)
+		(layer "F.Cu")
+		(net "VCC")
+	)
+	(segment
+		(start 142.145 119.205)
+		(end 142.225 119.285)
+		(width 0.1524)
+		(layer "F.Cu")
+		(net "/INPUT")
+	)
+	(segment
+		(start 136.2875 119.205)
+		(end 142.145 119.205)
+		(width 0.1524)
+		(layer "F.Cu")
+		(net "/INPUT")
+	)
+	(segment
+		(start 129.1125 117.935)
+		(end 126.985 117.935)
+		(width 0.1524)
+		(layer "F.Cu")
+		(net "Net-(D1-A)")
+	)
+	(segment
+		(start 126.985 117.935)
+		(end 125.715 119.205)
+		(width 0.1524)
+		(layer "F.Cu")
+		(net "Net-(D1-A)")
+	)
+	(segment
+		(start 142.225 121.11)
+		(end 141.59 121.11)
+		(width 0.1524)
+		(layer "F.Cu")
+		(net "Net-(J1-Pin_1)")
+	)
+	(segment
+		(start 141.59 121.11)
+		(end 135.24 127.46)
+		(width 0.1524)
+		(layer "F.Cu")
+		(net "Net-(J1-Pin_1)")
 	)
 	(zone
