File: tutorial-77.kicad_pcb (KiCad board)
At the start: 2 copper layers, 25 x 25 mm, 7 parts, among them J1 Conn_01x03_Pin, U1 ATtiny85-20S

Commit message: auto-router plan_b
Routing:
- net GND: track 0.00 -> 43.3 mm
- net Net-(D1-A): track 0.00 -> 15.9 mm
- net VCC: track 0.00 -> 12.3 mm
- net Net-(J1-Pin_1): track 0.00 -> 9.49 mm
- net /INPUT: track 0.00 -> 5.57 mm
- net Net-(D1-K): track 0.00 -> 2.53 mm
Changed lines of the file:
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@@
 		)
 	)
+	(segment
+		(start 140 115.5)
+		(end 140 117.925)
+		(width 0.1524)
+		(layer "F.Cu")
+		(net "Net-(D1-K)")
+	)
+	(segment
+		(start 140 117.925)
+		(end 139.925 118)
+		(width 0.1524)
+		(layer "F.Cu")
+		(net "Net-(D1-K)")
+	)
+	(segment
+		(start 142.5036 115.062854)
+		(end 142.237146 114.7964)
+		(width 0.1524)
+		(layer "F.Cu")
+		(net "GND")
+	)
+	(segment
+		(start 132.7 121.259598)
+		(end 129.929002 118.4886)
+		(width 0.1524)
+		(layer "F.Cu")
+		(net "GND")
+	)
+	(segment
+		(start 125.3886 116.1114)
+		(end 135.7339 116.1114)
+		(width 0.1524)
+		(layer "F.Cu")
+		(net "GND")
+	)
+	(segment
+		(start 142.5036 117.2464)
+		(end 142.5036 115.062854)
+		(width 0.1524)
+		(layer "F.Cu")
+		(net "GND")
+	)
+	(segment
+		(start 132.7 127.46)
+		(end 132.7 121.259598)
+		(width 0.1524)
+		(layer "F.Cu")
+		(net "GND")
+	)
+	(segment
+		(start 128.295998 116.1114)
+		(end 135.7339 116.1114)
+		(width 0.1524)
+		(layer "F.Cu")
+		(net "GND")
+	)
+	(segment
+		(start 141.75 118)
+		(end 142.5036 117.2464)
+		(width 0.1524)
+		(layer "F.Cu")
+		(net "GND")
+	)
+	(segment
+		(start 138.1561 114.7964)
+		(end 136.2875 116.665)
+		(width 0.1524)
+		(layer "F.Cu")
+		(net "GND")
+	)
+	(segment
+		(start 129.929002 118.4886)
+		(end 128.295998 118.4886)
+		(width 0.1524)
+		(layer "F.Cu")
+		(net "GND")
+	)
+	(segment
+		(start 128.0714 118.264002)
+		(end 128.0714 116.335998)
+		(width 0.1524)
+		(layer "F.Cu")
+		(net "GND")
+	)
+	(segment
+		(start 135.7339 116.1114)
+		(end 136.2875 116.665)
+		(width 0.1524)
+		(layer "F.Cu")
+		(net "GND")
+	)
+	(segment
+		(start 125.3625 116.1375)
+		(end 125.3886 116.1114)
+		(width 0.1524)
+		(layer "F.Cu")
+		(net "GND")
+	)
+	(segment
+		(start 128.0714 116.335998)
+		(end 128.295998 116.1114)
+		(width 0.1524)
+		(layer "F.Cu")
+		(net "GND")
+	)
+	(segment
+		(start 142.237146 114.7964)
+		(end 138.1561 114.7964)
+		(width 0.1524)
+		(layer "F.Cu")
+		(net "GND")
+	)
+	(segment
+		(start 128.295998 118.4886)
+		(end 128.0714 118.264002)
+		(width 0.1524)
+		(layer "F.Cu")
+		(net "GND")
+	)
+	(segment
+		(start 125.3625 117.8625)
+		(end 127.975 120.475)
+		(width 0.1524)
+		(layer "F.Cu")
+		(net "VCC")
+	)
+	(segment
+		(start 130.16 127.46)
+		(end 129.1125 126.4125)
+		(width 0.1524)
+		(layer "F.Cu")
+		(net "VCC")
+	)
+	(segment
+		(start 129.1125 126.4125)
+		(end 129.1125 120.475)
+		(width 0.1524)
+		(layer "F.Cu")
+		(net "VCC")
+	)
+	(segment
+		(start 127.975 120.475)
+		(end 129.1125 120.475)
+		(width 0.1524)
+		(layer "F.Cu")
+		(net "VCC")
+	)
+	(segment
+		(start 140.8214 119.1164)
+		(end 141.525 119.82)
+		(width 0.1524)
+		(layer "F.Cu")
+		(net "/INPUT")
+	)
+	(segment
+		(start 136.3761 119.1164)
+		(end 140.8214 119.1164)
+		(width 0.1524)
+		(layer "F.Cu")
+		(net "/INPUT")
+	)
+	(segment
+		(start 136.2875 119.205)
+		(end 136.3761 119.1164)
+		(width 0.1524)
+		(layer "F.Cu")
+		(net "/INPUT")
+	)
+	(segment
+		(start 140.6411 116.6089)
+		(end 140.6411 118.437146)
+		(width 0.1524)
+		(layer "F.Cu")
+		(net "Net-(D1-A)")
+	)
+	(segment
+		(start 140.6411 118.437146)
+		(end 140.374646 118.7036)
+		(width 0.1524)
+		(layer "F.Cu")
+		(net "Net-(D1-A)")
+	)
+	(segment
+		(start 137.990354 117.2186)
+		(end 129.8289 117.2186)
+		(width 0.1524)
+		(layer "F.Cu")
+		(net "Net-(D1-A)")
+	)
+	(segment
+		(start 141.75 115.5)
+		(end 140.6411 116.6089)
+		(width 0.1524)
+		(layer "F.Cu")
+		(net "Net-(D1-A)")
+	)
+	(segment
+		(start 140.374646 118.7036)
+		(end 139.475354 118.7036)
+		(width 0.1524)
+		(layer "F.Cu")
+		(net "Net-(D1-A)")
+	)
+	(segment
+		(start 139.475354 118.7036)
+		(end 137.990354 117.2186)
+		(width 0.1524)
+		(layer "F.Cu")
+		(net "Net-(D1-A)")
+	)
+	(segment
+		(start 129.8289 117.2186)
+		(end 129.1125 117.935)
+		(width 0.1524)
+		(layer "F.Cu")
+		(net "Net-(D1-A)")
+	)
+	(segment
+		(start 139.7 119.82)
+		(end 139.7 123)
+		(width 0.1524)
+		(layer "F.Cu")
+		(net "Net-(J1-Pin_1)")
+	)
+	(segment
+		(start 139.7 123)
+		(end 135.24 127.46)
+		(width 0.1524)
+		(layer "F.Cu")
+		(net "Net-(J1-Pin_1)")
+	)
 	(zone
 		(net "GND")
